File: hardware/KiCad/v1.4/SourceFIle.kicad_pcb (KiCad board)
At the start: 4 copper layers, 53 x 32 mm, 86 parts, among them IC1 ESP32-S3-WROOM-1-N16R2, IC5 ADS1115IRUGT, J1 10118192-0002LF, J2 Debug, J4 Screw_Terminal_01x03, SW1 SW_SPST, SW2 SW_SPST, U1 TPS630250RNCT, U2 MCP4725A3T-E/CH, U3 SN65HVD10DR, U4 IIS3DWBTR, U5 TSV912IQ2T, U6 ISM330DLCTR

Commit message: v1.41
fix the issue with PCB file
Parts:
- added R3: 10K, Resistor_SMD:R_0603_1608Metric_Pad0.98x0.95mm_HandSolder, F.Cu at (113.2, 71.0)
- added R7: 10K 0.2W, Resistor_SMD:R_0603_1608Metric_Pad0.98x0.95mm_HandSolder, F.Cu at (113.2, 75.5)
Connections:
- net /IO14 renamed /ESP32 S3/GPIO14
- C2 pad 2: Earth -> Net-(U1-FB)
- C3 pad 2: Earth -> Net-(U1-FB)
- IC1 pad 10: /D_MAIN -> /ESP32 S3/GPIO17
- IC1 pad 11: /R_MAIN -> /ESP32 S3/GPIO18
- IC1 pad 12: /SDA -> /ESP32 S3/GPIO8
- IC1 pad 17: /SCL -> /ESP32 S3/GPIO9
- IC1 pad 18: /CS -> /ESP32 S3/GPIO10
- IC1 pad 19: /MOSI -> /ESP32 S3/GPIO11
- IC1 pad 20: /CLK -> /ESP32 S3/GPIO12
- IC1 pad 21: /MISO -> /ESP32 S3/GPIO13
- IC1 pad 28: /ESP32 S3/GPIO35 -> /SCK
- IC1 pad 29: /ESP32 S3/GPIO36 -> /CS0
- IC1 pad 30: /ESP32 S3/GPIO37 -> /MOSI
- IC1 pad 31: /ESP32 S3/GPIO38 -> /MISO
- IC1 pad 38: /IO2 -> /ESP32 S3/GPIO2
- IC1 pad 39: /DE_MAIN -> /ESP32 S3/GPIO1
- IC1 pad 7: /IO7 -> /ESP32 S3/GPIO7
- IC1 pad 9: /IO16 -> /IO15
- R2 pad 1: Earth -> Net-(U1-FB)
- R2 pad 2: Net-(U1-FB) -> Earth
- R28 pad 2: Net-(U6-SDO/SAO) -> unconnected-(R28-Pad2)
- U6 pad 1: Net-(U6-SDO/SAO) -> /MISO
- U6 pad 12: Net-(U6-CS) -> /CS0
- U6 pad 13: /SCL -> /SCK
- U6 pad 14: /SDA -> /MOSI
- U6 pad 9: /IO16 -> /IO15
Routing:
- net +3.3V: track 345.3 -> 0.00 mm
- net Earth: track 291.5 -> 0.00 mm, vias 41 -> 40
- net /SDA: track 97.8 -> 0.00 mm, vias 6 -> 0
- net /SCL: track 73.0 -> 0.00 mm
- net /ESP32 S3/GPIO0: track 66.0 -> 0.00 mm
- net /ESP32 S3/CHIP_PU: track 64.0 -> 0.00 mm
- net /MOSI: track 49.9 -> 0.00 mm, vias 2 -> 8
- net /CS: track 49.7 -> 0.00 mm
- net /CLK: track 49.7 -> 0.00 mm
- net /MISO: track 49.7 -> 0.00 mm, vias 2 -> 3
- net /D+: track 43.5 -> 0.00 mm
- net /D-: track 42.1 -> 0.00 mm
- net /IO7: track 40.8 -> 0.00 mm
- net /IO16: track 39.0 -> 0.00 mm, vias 2 -> 0
- net /IO15: track 37.4 -> 0.00 mm, vias 2 -> 4
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